Commit message: rk

File: rossem_ws/src/Manipulator/my_xarm_lite6/my_lite6_description/urdf/lite6_robot.urdf.xacro (robot description, xacro)
@@ -1,4 +1,4 @@
 <?xml version="1.0"?>
-<robot xmlns:xacro="http://wiki.ros.org/xacro" name="lite6_robot">
+<robot xmlns:xacro="http://www.ros.org/wiki/xacro" name="lite6_robot">
   <!--
   <xacro:arg name="prefix" default="arm_"/>
@@ -42,4 +42,5 @@
   <xacro:arg name="mesh_suffix" default="stl"/>
   <xacro:arg name="kinematics_suffix" default=""/>
+  <xacro:include filename="$(find my_lite6_description)/urdf/depthai_macro.urdf.xacro" />
   <!-- load xarm device -->
   <xacro:include filename="$(find xarm_description)/urdf/xarm_device_macro.xacro" />
@@ -212,5 +213,5 @@
   <parent link="mountingplate_link"/>
   <child link="transportband_link"/>
-  <origin xyz="0.08 -0.15 0" rpy="1.57 0 0"/>
+  <origin xyz="0.005 -0.11 0" rpy="1.57 0 0"/>
 </joint>
 <!-- camera link -->
@@ -244,5 +245,5 @@
   <parent link="mountingplate_link"/>
   <child link="camera_compleet_link"/>
-  <origin xyz="0.4 -0.3 0" rpy="0 0 3.14"/>
+  <origin xyz="0.19 -0.245 -0.02" rpy="0 0 3.14"/>
 </joint>
 <!-- Schroevendraaier link
@@ -342,4 +343,18 @@
   <origin xyz="-0.115 -0.04 -0.05" rpy="0 0 0"/> <!-- pas aan voor juiste positie -->
 </joint>
+<!-- camera position -->
+<!-- DepthAI-camera toevoegen aan robot -->
+<xacro:depthai_camera
+  camera_name="oak_camera"
+  camera_model="OAK-D"
+  parent="world"
+  base_frame="camera_link"
+  cam_pos_x="-0.14"
+  cam_pos_y="-0.26"
+  cam_pos_z="0.54"
+  cam_roll="0.0"
+  cam_pitch="1.5708"
+  cam_yaw="-1.5708"
+/>
 </robot>
 <!--

Commit message: sweet spot

File: rossem_ws/src/Manipulator/my_xarm_lite6/my_lite6_description/urdf/lite6_robot.urdf.xacro (robot description, xacro)
@@ -213,5 +213,5 @@
   <parent link="mountingplate_link"/>
   <child link="transportband_link"/>
-  <origin xyz="0.005 -0.11 0" rpy="1.57 0 0"/>
+  <origin xyz="0.005 -0.11 -0.04" rpy="1.57 0 0"/>
 </joint>
 <!-- camera link -->
@@ -352,5 +352,5 @@
   cam_pos_x="-0.14"
   cam_pos_y="-0.26"
-  cam_pos_z="0.54"
+  cam_pos_z="0.61"
   cam_roll="0.0"
   cam_pitch="1.5708"

Commit message: gtgf

File: rossem_ws/src/Manipulator/my_xarm_lite6/my_lite6_description/urdf/lite6_robot.urdf.xacro (robot description, xacro)
@@ -343,4 +343,36 @@
   <origin xyz="-0.115 -0.04 -0.05" rpy="0 0 0"/> <!-- pas aan voor juiste positie -->
 </joint>
+<!-- bovenplaat -->
+<link name="bovenplaat_link">
+  <visual>
+    <origin xyz="0 0 0.01" rpy="0 0 0"/>
+    <geometry>
+      <mesh filename="package://my_lite6_description/meshes/bovenplaat.STL" scale="0.001 0.001 0.001"/>
+    </geometry>
+    <material name="gray">
+      <color rgba="0.5 0.5 0.5 1.0"/>
+    </material>
+  </visual>
+  <collision>
+    <origin xyz="0 0 0" rpy="0 0 0"/>
+    <geometry>
+      <mesh filename="package://my_lite6_description/meshes/bovenplaat.STL" scale="0.001 0.001 0.001"/>
+    </geometry>
+  </collision>
+  <inertial>
+    <mass value="0.3892"/>
+    <origin xyz="-0.11546 0.09763 0.06783" rpy="0 0 0"/>
+    <inertia
+      ixx="0.01311039287" ixy="-0.00770441053" ixz="-0.00641160864"
+      iyy="0.04087287606" iyz="0.00479622192"
+      izz="0.042905365"/>
+  </inertial>
+</link>
+<!-- bovenplaat -->
+<joint name="mountingplate_to_bovenplaat_joint" type="fixed">
+  <parent link="mountingplate_link"/>
+  <child link="bovenplaat_link"/>
+  <origin xyz="0.39 0.25 0.7" rpy="0 0 3.14"/>
+</joint>
 <!-- camera position -->
 <!-- DepthAI-camera toevoegen aan robot -->
